File: pcb/v2/roBa_L/roba_L.kicad_pcb (KiCad board)
At the start: 2 copper layers, 123.9 x 94.5 mm, 56 parts, among them J1 Conn_01x01-Connector_Generic, J2 Conn_01x01-Connector_Generic, J3 Conn_01x01-Connector_Generic, J4 Conn_01x01-Connector_Generic, J5 Conn_01x01-Connector_Generic, J6 Conn_01x01-Connector_Generic, J7 Conn_01x01-Connector_Generic, SW1 SW_PUSH, SW10 SW_PUSH, SW11 SW_PUSH, SW12 SW_PUSH, SW13 SW_PUSH, SW14 SW_PUSH, SW15 SW_PUSH, SW16 SW_PUSH, SW17 SW_PUSH, SW18 SW_PUSH, SW19 SW_PUSH, SW2 SW_PUSH, SW20 SW_PUSH, SW21 RotaryEncoder_Switch, SW22 SW_PUSH, SW23 SW_PUSH, SW24 SW_SPDT, SW3 SW_PUSH, SW4 SW_PUSH, SW5 SW_PUSH, SW6 SW_PUSH, SW7 SW_PUSH, SW8 SW_PUSH, SW9 SW_PUSH

Commit message: Update left PCB
Parts:
- SW1, SW10, SW11, SW12, SW13, SW14, SW15, SW17, SW18, SW19, SW2, SW22, SW3, SW4, SW5, SW6, SW7, SW8, SW9: footprint roBa:SW_MX -> roBa:gateron-ks27-choc-v1-mx-hotswap-curved-pads
- SW16, SW20, SW23: footprint roBa:SW_MX_Choc -> roBa:gateron-ks27-choc-v1-mx-hotswap-curved-pads
- SW21: footprint roBa:SW_MX_EC12 -> roBa:gateron-ks27-choc-v1-mx-hotswap-ec12
- moved D23 13.7 mm to (184.6, 114.6)
- moved D20 7.56 mm to (172.5, 114.4)
- moved D16 7.42 mm to (148.8, 113.5)
- turned SW16 to 180 degrees
- turned SW20 to 171 degrees
- turned SW23 to 160 degrees
Connections:
- SW1 pad 1: Col0 -> Net-(D1-A)
- SW1 pad 2: Net-(D1-A) -> Col0
- SW10 pad 1: Col2 -> Net-(D10-A)
- SW10 pad 2: Net-(D10-A) -> Col2
- SW11 pad 1: Col2 -> Net-(D11-A)
- SW11 pad 2: Net-(D11-A) -> Col2
- SW12 pad 1: Col2 -> Net-(D12-A)
- SW12 pad 2: Net-(D12-A) -> Col2
- SW13 pad 1: Col3 -> Net-(D13-A)
- SW13 pad 2: Net-(D13-A) -> Col3
- SW14 pad 1: Col3 -> Net-(D14-A)
- SW14 pad 2: Net-(D14-A) -> Col3
- SW15 pad 1: Col3 -> Net-(D15-A)
- SW15 pad 2: Net-(D15-A) -> Col3
- SW16 pad 1: Col3 -> Net-(D16-A)
- SW16 pad 2: Net-(D16-A) -> Col3
- SW17 pad 1: Col4 -> Net-(D17-A)
- SW17 pad 2: Net-(D17-A) -> Col4
- SW18 pad 1: Col4 -> Net-(D18-A)
- SW18 pad 2: Net-(D18-A) -> Col4
- SW19 pad 1: Col4 -> Net-(D19-A)
- SW19 pad 2: Net-(D19-A) -> Col4
- SW2 pad 1: Col0 -> Net-(D2-A)
- SW2 pad 2: Net-(D2-A) -> Col0
- SW20 pad 1: Col4 -> Net-(D20-A)
- SW20 pad 2: Net-(D20-A) -> Col4
- SW21 pad 2: Col5 -> Net-(D21-A)
- SW22 pad 1: Col5 -> Net-(D22-A)
- SW22 pad 2: Net-(D22-A) -> Col5
- SW23 pad 1: Col5 -> Net-(D23-A)
- SW23 pad 2: Net-(D23-A) -> Col5
- SW3 pad 1: Col0 -> Net-(D3-A)
- SW3 pad 2: Net-(D3-A) -> Col0
- SW4 pad 1: Col0 -> Net-(D4-A)
- SW4 pad 2: Net-(D4-A) -> Col0
- SW5 pad 1: Col1 -> Net-(D5-A)
- SW5 pad 2: Net-(D5-A) -> Col1
- SW6 pad 1: Col1 -> Net-(D6-A)
- SW6 pad 2: Net-(D6-A) -> Col1
- SW7 pad 1: Col1 -> Net-(D7-A)
- SW7 pad 2: Net-(D7-A) -> Col1
- SW8 pad 1: Col1 -> Net-(D8-A)
- SW8 pad 2: Net-(D8-A) -> Col1
- SW9 pad 1: Col2 -> Net-(D9-A)
- SW9 pad 2: Net-(D9-A) -> Col2
- U1 pad 12: unconnected-(U1-3V3-Pad12) -> VCC
- U1 pad 14: VCC -> unconnected-(U1-5V-Pad14)
Routing:
- net Row3: track 201.8 -> 160.2 mm, vias 2 -> 4
- net Col5: track 85.6 -> 67.4 mm, vias 0 -> 2
- net Col4: track 126.1 -> 110.3 mm, vias 1 -> 2
- net Net-(D23-A): track 12.8 -> 26.3 mm
- net Net-(B1--): track 40.6 -> 53.8 mm
- net Row2: track 177.2 -> 167.3 mm
- net Row0: track 122.6 -> 114.7 mm, vias 5 -> 7
- net GND: track 80.6 -> 74.7 mm, vias 2 -> 0
- net Col3: track 173.6 -> 169.5 mm
- net Net-(D21-A): track 25.4 -> 29.4 mm
- net Col2: track 148.6 -> 152.3 mm
- net RE_A1: track 18.1 -> 14.6 mm
- net Bat: track 14.2 -> 11.0 mm
- net Net-(D15-A): track 16.4 -> 13.3 mm
- net Net-(D14-A): track 16.3 -> 13.3 mm
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
Commit message: Update schematics and PCBs
Parts:
- D1, D10, D11, D12, D13, D14, D15, D16, D17, D18, D19, D2, D20, D21, D22, D23, D3, D4, D5, D6, D7, D8, D9: footprint roBa:Diode_SMD -> Diode_SMD:D_SOD-123; moved to B.Cu
- moved D15 11.0 mm to (153.5, 92.4)
- moved D21 2.98 mm to (191.1, 90.6)
- moved D20 2.81 mm to (175.3, 114.9), turned to 0 degrees
- moved D22 2.79 mm to (190.9, 110.2)
- moved D12 2.78 mm to (134.5, 119.8)
- moved D18 2.78 mm to (172.6, 86.4)
- moved D1 2.75 mm to (96.4, 73.9)
- moved D6 2.75 mm to (115.4, 86.4)
- moved D16 2.75 mm to (151.6, 113.5)
- moved D10 2.73 mm to (134.4, 81.6)
- moved D3 2.73 mm to (96.3, 112.1)
- moved D19 2.70 mm to (172.5, 105.5)
- moved D4 2.70 mm to (96.3, 131.1)
- moved D7 2.70 mm to (115.4, 105.4)
- moved D14 2.70 mm to (153.5, 84.0)
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Connections:
- SW15 pad 1: Net-(D15-A) -> Col3
- SW15 pad 2: Col3 -> Net-(D15-A)
Routing:
- net Row2: track 167.3 -> 182.4 mm
- net Col1: track 160.7 -> 163.5 mm
- net Col0: track 187.1 -> 184.5 mm
- net Col2: track 152.3 -> 154.7 mm
- net Net-(D23-A): track 26.3 -> 28.0 mm
- net Net-(D20-A): track 13.4 -> 15.0 mm
- net Row3: track 160.2 -> 159.6 mm
- net Net-(D15-A): track 13.3 -> 14.0 mm
- net Net-(B1--): track 53.8 -> 53.2 mm
- net GND: track 74.7 -> 74.4 mm, vias 0 -> 1
