File: pcb/v2/roBa_L/roba_L.kicad_sch (KiCad schematic)
At the start: 56 parts, among them J1 Conn_01x01-Connector_Generic, J2 Conn_01x01-Connector_Generic, J3 Conn_01x01-Connector_Generic, J4 Conn_01x01-Connector_Generic, J5 Conn_01x01-Connector_Generic, J6 Conn_01x01-Connector_Generic, J7 Conn_01x01-Connector_Generic, SW1 SW_PUSH, SW10 SW_PUSH, SW11 SW_PUSH, SW12 SW_PUSH, SW13 SW_PUSH, SW14 SW_PUSH, SW15 SW_PUSH, SW16 SW_PUSH, SW17 SW_PUSH, SW18 SW_PUSH, SW19 SW_PUSH, SW2 SW_PUSH, SW20 SW_PUSH, SW21 RotaryEncoder_Switch, SW22 SW_PUSH, SW23 SW_PUSH, SW24 SW_SPDT, SW3 SW_PUSH, SW4 SW_PUSH, SW5 SW_PUSH, SW6 SW_PUSH, SW7 SW_PUSH, SW8 SW_PUSH, SW9 SW_PUSH

Commit message: Update left PCB
Parts:
- SW1, SW10, SW11, SW12, SW13, SW14, SW15, SW17, SW18, SW19, SW2, SW22, SW3, SW4, SW5, SW6, SW7, SW8, SW9: footprint roBa:SW_MX -> roBa:gateron-ks27-choc-v1-mx-hotswap-curved-pads
- SW16, SW20, SW23: footprint roBa:SW_MX_Choc -> roBa:gateron-ks27-choc-v1-mx-hotswap-curved-pads
- SW21: footprint roBa:SW_MX_EC12 -> roBa:gateron-ks27-choc-v1-mx-hotswap-ec12
Connections:
- net Col0: now also SW1.2, SW2.2, SW3.2, SW4.2; no longer SW1.1, SW2.1, SW3.1, SW4.1
- net Col1: now also SW5.2, SW6.2, SW7.2, SW8.2; no longer SW5.1, SW6.1, SW7.1, SW8.1
- net Col2: now also SW10.2, SW11.2, SW12.2, SW9.2; no longer SW10.1, SW11.1, SW12.1, SW9.1
- net Col3: now also SW13.2, SW14.2, SW15.2, SW16.2; no longer SW13.1, SW14.1, SW15.1, SW16.1
- net Col4: now also SW17.2, SW18.2, SW19.2, SW20.2; no longer SW17.1, SW18.1, SW19.1, SW20.1
- net Col5: now also SW22.2, SW23.2; no longer SW22.1, SW23.1
- net VCC: now also U1.12 (3V3); no longer U1.14 (5V)
- net at D6.2 (A): now also SW6.1; no longer SW6.2
- net at D9.2 (A): now also SW9.1; no longer SW9.2
- net at D22.2 (A): now also SW22.1; no longer SW22.2
- net at D8.2 (A): now also SW8.1; no longer SW8.2
- net at D10.2 (A): now also SW10.1; no longer SW10.2
- net at D5.2 (A): now also SW5.1; no longer SW5.2
- net at D13.2 (A): now also SW13.1; no longer SW13.2
- net at D3.2 (A): now also SW3.1; no longer SW3.2
- net at D2.2 (A): now also SW2.1; no longer SW2.2
- net at D11.2 (A): now also SW11.1; no longer SW11.2
- net at D7.2 (A): now also SW7.1; no longer SW7.2
- net at D12.2 (A): now also SW12.1; no longer SW12.2
- net at D20.2 (A): now also SW20.1; no longer SW20.2
- net at D1.2 (A): now also SW1.1; no longer SW1.2
- net at D16.2 (A): now also SW16.1; no longer SW16.2
- net at D23.2 (A): now also SW23.1; no longer SW23.2
- net at D14.2 (A): now also SW14.1; no longer SW14.2
- net at D19.2 (A): now also SW19.1; no longer SW19.2
- net at D15.2 (A): now also SW15.1; no longer SW15.2
- net at D17.2 (A): now also SW17.1; no longer SW17.2
- net at D18.2 (A): now also SW18.1; no longer SW18.2
- net at D4.2 (A): now also SW4.1; no longer SW4.2

Commit message: Update schematics and PCBs
Parts:
- D1, D10, D11, D12, D13, D14, D15, D16, D17, D18, D19, D2, D20, D21, D22, D23, D3, D4, D5, D6, D7, D8, D9: footprint roBa:Diode_SMD -> Diode_SMD:D_SOD-123
Connections:
- net VCC renamed +3.3V
Changed lines of the file:
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@@
 			)
 		)
-		(property "Footprint" "roBa:Diode_SMD"
+		(property "Footprint" "Diode_SMD:D_SOD-123"
 			(at 149.86 72.39 0)
 			(effects
@@
 	)
 	(symbol
-		(lib_id "power:VCC")
-		(at 99.06 73.66 270)
-		(unit 1)
-		(exclude_from_sim no)
-		(in_bom yes)
-		(on_board yes)
-		(dnp no)
-		(property "Reference" "#PWR05"
-			(at 95.25 73.66 0)
-			(effects
-				(font
-					(size 1.27 1.27)
-				)
-				(hide yes)
-			)
-		)
-		(property "Value" "VCC"
-			(at 103.4542 74.0918 0)
-			(effects
-				(font
-					(size 1.27 1.27)
-				)
-			)
-		)
-		(property "Footprint" ""
-			(at 99.06 73.66 0)
-			(effects
-				(font
-					(size 1.27 1.27)
-				)
-				(hide yes)
-			)
-		)
-		(property "Datasheet" ""
-			(at 99.06 73.66 0)
-			(effects
-				(font
-					(size 1.27 1.27)
-				)
-				(hide yes)
-			)
-		)
-		(property "Description" ""
-			(at 99.06 73.66 0)
-			(effects
-				(font
-					(size 1.27 1.27)
-				)
-				(hide yes)
-			)
-		)
-		(pin "1"
-		)
-		(instances
-			(project "roba_L"
-				(path "/10ebe2a9-954f-43ec-9eb9-ae4cbd386108"
-					(reference "#PWR05")
-					(unit 1)
-				)
-			)
-		)
-	)
-	(symbol
 		(lib_id "Device:D")
 		(at 168.91 53.34 270)
@@
 			)
 		)
-		(property "Footprint" "roBa:Diode_SMD"
+		(property "Footprint" "Diode_SMD:D_SOD-123"
 			(at 168.91 53.34 0)
 			(effects
@@
 			)
 		)
-		(property "Footprint" "roBa:Diode_SMD"
+		(property "Footprint" "Diode_SMD:D_SOD-123"
 			(at 226.06 91.44 0)
 			(effects
@@
 			)
 		)
-		(property "Footprint" "roBa:Diode_SMD"
+		(property "Footprint" "Diode_SMD:D_SOD-123"
 			(at 149.86 109.22 0)
 			(effects
@@
 			)
 		)
-		(property "Footprint" "roBa:Diode_SMD"
+		(property "Footprint" "Diode_SMD:D_SOD-123"
 			(at 168.91 72.39 0)
 			(effects
@@
 			)
 		)
-		(property "Footprint" "roBa:Diode_SMD"
+		(property "Footprint" "Diode_SMD:D_SOD-123"
 			(at 226.06 72.39 0)
 			(effects
@@
 			)
 		)
-		(property "Footprint" "roBa:Diode_SMD"
+		(property "Footprint" "Diode_SMD:D_SOD-123"
 			(at 149.86 53.34 0)
 			(effects
@@
 			)
 		)
-		(property "Footprint" "roBa:Diode_SMD"
+		(property "Footprint" "Diode_SMD:D_SOD-123"
 			(at 130.81 91.44 0)
 			(effects
@@
 	)
 	(symbol
-		(lib_id "power:VCC")
-		(at 111.76 167.64 0)
-		(unit 1)
-		(exclude_from_sim no)
-		(in_bom yes)
-		(on_board yes)
-		(dnp no)
-		(property "Reference" "#PWR07"
-			(at 111.76 171.45 0)
-			(effects
-				(font
-					(size 1.27 1.27)
-				)
-				(hide yes)
-			)
-		)
-		(property "Value" "VCC"
-			(at 112.1918 163.2458 0)
-			(effects
-				(font
-					(size 1.27 1.27)
-				)
-			)
-		)
-		(property "Footprint" ""
-			(at 111.76 167.64 0)
-			(effects
-				(font
-					(size 1.27 1.27)
-				)
-				(hide yes)
-			)
-		)
-		(property "Datasheet" ""
-			(at 111.76 167.64 0)
-			(effects
-				(font
-					(size 1.27 1.27)
-				)
-				(hide yes)
-			)
-		)
-		(property "Description" ""
-			(at 111.76 167.64 0)
-			(effects
-				(font
-					(size 1.27 1.27)
-				)
-				(hide yes)
-			)
-		)
-		(pin "1"
-		)
-		(instances
-			(project "roba_L"
-				(path "/10ebe2a9-954f-43ec-9eb9-ae4cbd386108"
-					(reference "#PWR07")
-					(unit 1)
-				)
-			)
-		)
-	)
-	(symbol
 		(lib_id "power:GND")
 		(at 45.72 171.45 0)
@@
 			)
 		)
-		(property "Footprint" "roBa:Diode_SMD"
+		(property "Footprint" "Diode_SMD:D_SOD-123"
 			(at 207.01 109.22 0)
 			(effects
@@
 			)
 		)
-		(property "Footprint" "roBa:Diode_SMD"
+		(property "Footprint" "Diode_SMD:D_SOD-123"
 			(at 130.81 53.34 0)
 			(effects
@@
 			)
 		)
-		(property "Footprint" "roBa:Diode_SMD"
+		(property "Footprint" "Diode_SMD:D_SOD-123"
 			(at 226.06 109.22 0)
 			(effects
@@
 	)
 	(symbol
+		(lib_id "power:+3.3V")
+		(at 111.76 167.64 0)
+		(unit 1)
+		(exclude_from_sim no)
+		(in_bom yes)
+		(on_board yes)
+		(dnp no)
+		(fields_autoplaced yes)
+		(property "Reference" "#PWR05"
+			(at 111.76 171.45 0)
+			(effects
+				(font
+					(size 1.27 1.27)
+				)
+				(hide yes)
+			)
+		)
+		(property "Value" "+3.3V"
+			(at 111.76 162.56 0)
+			(effects
+				(font
+					(size 1.27 1.27)
+				)
+			)
+		)
+		(property "Footprint" ""
+			(at 111.76 167.64 0)
+			(effects
+				(font
+					(size 1.27 1.27)
+				)
+				(hide yes)
+			)
+		)
+		(property "Datasheet" ""
+			(at 111.76 167.64 0)
+			(effects
+				(font
+					(size 1.27 1.27)
+				)
+				(hide yes)
+			)
+		)
+		(property "Description" "Power symbol creates a global label with name \"+3.3V\""
+			(at 111.76 167.64 0)
+			(effects
+				(font
+					(size 1.27 1.27)
+				)
+				(hide yes)
+			)
+		)
+		(pin "1"
+		)
+		(instances
+			(project "roba_L"
+				(path "/10ebe2a9-954f-43ec-9eb9-ae4cbd386108"
+					(reference "#PWR05")
+					(unit 1)
+				)
+			)
+		)
+	)
+	(symbol
 		(lib_id "Device:D")
 		(at 187.96 72.39 270)
@@
 			)
 		)
-		(property "Footprint" "roBa:Diode_SMD"
+		(property "Footprint" "Diode_SMD:D_SOD-123"
 			(at 187.96 72.39 0)
 			(effects
@@
 			)
 		)
-		(property "Footprint" "roBa:Diode_SMD"
+		(property "Footprint" "Diode_SMD:D_SOD-123"
 			(at 207.01 91.44 0)
 			(effects
@@
 			)
 		)
-		(property "Footprint" "roBa:Diode_SMD"
+		(property "Footprint" "Diode_SMD:D_SOD-123"
 			(at 187.96 91.44 0)
 			(effects
@@
 			)
 		)
-		(property "Footprint" "roBa:Diode_SMD"
+		(property "Footprint" "Diode_SMD:D_SOD-123"
 			(at 168.91 109.22 0)
 			(effects
@@
 			)
 		)
-		(property "Footprint" "roBa:Diode_SMD"
+		(property "Footprint" "Diode_SMD:D_SOD-123"
 			(at 130.81 72.39 0)
 			(effects
@@
 			)
 		)
-		(property "Footprint" "roBa:Diode_SMD"
+		(property "Footprint" "Diode_SMD:D_SOD-123"
 			(at 207.01 72.39 0)
 			(effects
@@
 			)
 		)
-		(property "Footprint" "roBa:Diode_SMD"
+		(property "Footprint" "Diode_SMD:D_SOD-123"
 			(at 149.86 91.44 0)
 			(effects
@@
 			)
 		)
-		(property "Footprint" "roBa:Diode_SMD"
+		(property "Footprint" "Diode_SMD:D_SOD-123"
 			(at 187.96 53.34 0)
 			(effects
@@
 			)
 		)
-		(property "Footprint" "roBa:Diode_SMD"
+		(property "Footprint" "Diode_SMD:D_SOD-123"
 			(at 130.81 109.22 0)
 			(effects
@@
 			)
 		)
-		(property "Footprint" "roBa:Diode_SMD"
+		(property "Footprint" "Diode_SMD:D_SOD-123"
 			(at 187.96 109.22 0)
 			(effects
@@
 	)
 	(symbol
+		(lib_id "power:+3.3V")
+		(at 99.06 73.66 270)
+		(unit 1)
+		(exclude_from_sim no)
+		(in_bom yes)
+		(on_board yes)
+		(dnp no)
+		(fields_autoplaced yes)
+		(property "Reference" "#PWR02"
+			(at 95.25 73.66 0)
+			(effects
+				(font
+					(size 1.27 1.27)
+				)
+				(hide yes)
+			)
+		)
+		(property "Value" "+3.3V"
+			(at 102.87 73.6599 90)
+			(effects
+				(font
+					(size 1.27 1.27)
+				)
+				(justify left)
+			)
+		)
+		(property "Footprint" ""
+			(at 99.06 73.66 0)
+			(effects
+				(font
+					(size 1.27 1.27)
+				)
+				(hide yes)
+			)
+		)
+		(property "Datasheet" ""
+			(at 99.06 73.66 0)
+			(effects
+				(font
+					(size 1.27 1.27)
+				)
+				(hide yes)
+			)
+		)
+		(property "Description" "Power symbol creates a global label with name \"+3.3V\""
+			(at 99.06 73.66 0)
+			(effects
+				(font
+					(size 1.27 1.27)
+				)
+				(hide yes)
+			)
+		)
+		(pin "1"
+		)
+		(instances
+			(project ""
+				(path "/10ebe2a9-954f-43ec-9eb9-ae4cbd386108"
+					(reference "#PWR02")
+					(unit 1)
+				)
+			)
+		)
+	)
+	(symbol
 		(lib_id "Device:D")
 		(at 207.01 53.34 270)
@@
 			)
 		)
-		(property "Footprint" "roBa:Diode_SMD"
+		(property "Footprint" "Diode_SMD:D_SOD-123"
 			(at 207.01 53.34 0)
 			(effects
@@
 			)
 		)
-		(property "Footprint" "roBa:Diode_SMD"
+		(property "Footprint" "Diode_SMD:D_SOD-123"
 			(at 168.91 91.44 0)
 			(effects
