File: pcb/v2/roBa_R/roba_R.kicad_pcb (KiCad board)
At the start: 2 copper layers, 123.9 x 94.5 mm, 50 parts, among them J2 Conn_01x01-Connector_Generic, J3 Conn_01x01-Connector_Generic, J4 Conn_01x01-Connector_Generic, J5 Conn_01x01-Connector_Generic, J6 Conn_01x01-Connector_Generic, J7 Conn_01x01-Connector_Generic, SW1 SW_PUSH, SW10 SW_PUSH, SW11 SW_PUSH, SW12 SW_PUSH, SW13 SW_PUSH, SW14 SW_PUSH, SW15 SW_PUSH, SW16 SW_PUSH, SW17 SW_PUSH, SW18 SW_PUSH, SW19 SW_PUSH, SW2 SW_PUSH, SW20 SW_PUSH, SW21 SW_SPDT, SW3 SW_PUSH, SW4 SW_PUSH, SW5 SW_PUSH, SW6 SW_PUSH, SW7 SW_PUSH, SW8 SW_PUSH, SW9 SW_PUSH

Commit message: Update schematics and PCBs
Parts:
- removed D20: D, roBa:Diode_SMD
- removed J1: ~, roBa:pmw3610_connector
- removed SW20: SW_PUSH, roBa:SW_MX
- added J8: ~, vik:vik-keyboard-connector-horizontal, F.Cu at (206.1, 131.7)
- D1, D10, D11, D12, D13, D14, D15, D16, D17, D18, D19, D2, D3, D4, D5, D6, D7, D8, D9: footprint roBa:Diode_SMD -> Diode_SMD:D_SOD-123; moved to B.Cu
- SW1, SW10, SW11, SW13, SW14, SW15, SW17, SW18, SW19, SW2, SW3, SW4, SW5, SW6, SW7, SW8, SW9: footprint roBa:SW_MX -> roBa:gateron-ks27-choc-v1-mx-hotswap-curved-pads
- SW12, SW16: footprint roBa:SW_MX_Choc -> roBa:gateron-ks27-choc-v1-mx-hotswap-curved-pads
- moved D12 24.1 mm to (112.0, 124.0), turned to 10 degrees
- moved D16 12.8 mm to (122.9, 122.3)
- moved D17 2.88 mm to (205.4, 81.5)
- moved D19 2.86 mm to (205.4, 119.6)
- moved D1 2.83 mm to (129.2, 74.8)
- moved D18 2.81 mm to (205.4, 100.6)
- moved D3 2.81 mm to (129.2, 112.9)
- moved D7 2.76 mm to (148.2, 110.4)
- moved D6 2.76 mm to (148.2, 91.4)
- moved D5 2.76 mm to (148.2, 72.5)
- moved D11 2.76 mm to (167.2, 108.2)
- moved D9 2.73 mm to (167.2, 70.0)
- moved D10 2.73 mm to (167.2, 89.2)
- moved D13 2.73 mm to (186.2, 74.8)
- moved D15 2.73 mm to (186.2, 112.9)
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Connections:
- SW1 pad 1: Col0 -> Net-(D1-A)
- SW1 pad 2: Net-(D1-A) -> Col0
- SW10 pad 1: Col2 -> Net-(D10-A)
- SW10 pad 2: Net-(D10-A) -> Col2
- SW11 pad 1: Col2 -> Net-(D11-A)
- SW11 pad 2: Net-(D11-A) -> Col2
- SW12 pad 1: Col2 -> Net-(D12-A)
- SW12 pad 2: Net-(D12-A) -> Col2
- SW13 pad 1: Col3 -> Net-(D13-A)
- SW13 pad 2: Net-(D13-A) -> Col3
- SW14 pad 1: Col3 -> Net-(D14-A)
- SW14 pad 2: Net-(D14-A) -> Col3
- SW15 pad 1: Col3 -> Net-(D15-A)
- SW15 pad 2: Net-(D15-A) -> Col3
- SW16 pad 1: Col3 -> Net-(D16-A)
- SW16 pad 2: Net-(D16-A) -> Col3
- SW17 pad 1: Col4 -> Net-(D17-A)
- SW17 pad 2: Net-(D17-A) -> Col4
- SW18 pad 1: Col4 -> Net-(D18-A)
- SW18 pad 2: Net-(D18-A) -> Col4
- SW19 pad 1: Col4 -> Net-(D19-A)
- SW19 pad 2: Net-(D19-A) -> Col4
- SW2 pad 1: Col0 -> Net-(D2-A)
- SW2 pad 2: Net-(D2-A) -> Col0
- SW3 pad 1: Col0 -> Net-(D3-A)
- SW3 pad 2: Net-(D3-A) -> Col0
- SW4 pad 1: Col0 -> Net-(D4-A)
- SW4 pad 2: Net-(D4-A) -> Col0
- SW5 pad 1: Col1 -> Net-(D5-A)
- SW5 pad 2: Net-(D5-A) -> Col1
- SW6 pad 1: Col1 -> Net-(D6-A)
- SW6 pad 2: Net-(D6-A) -> Col1
- SW7 pad 1: Col1 -> Net-(D7-A)
- SW7 pad 2: Net-(D7-A) -> Col1
- SW8 pad 1: Col1 -> Net-(D8-A)
- SW8 pad 2: Net-(D8-A) -> Col1
- SW9 pad 1: Col2 -> Net-(D9-A)
- SW9 pad 2: Net-(D9-A) -> Col2
- U1 pad 12: 3.3V -> +3.3V
- U1 pad 14: VCC -> unconnected-(U1-5V-Pad14)
Routing:
- net Row3: track 249.7 -> 75.4 mm, vias 7 -> 2
- net +3.3V: track 0.00 -> 161.6 mm, vias 0 -> 8
- net 3.3V: track 149.3 -> 0.00 mm, vias 3 -> 0
- net CS: track 111.9 -> 137.7 mm, vias 3 -> 2
- net SCLK: track 125.1 -> 148.2 mm, vias 4 -> 3
- net Net-(D20-A): track 17.2 -> 0.00 mm
- net Col4: track 143.9 -> 129.0 mm
- net Row0: track 134.2 -> 120.9 mm, vias 8 -> 9
- net GND: track 173.8 -> 186.5 mm, vias 1 -> 2
- net MOTION: track 153.2 -> 163.7 mm, vias 4 -> 5
- net Col2: track 172.6 -> 181.9 mm
- net Row2: track 153.3 -> 161.0 mm, vias 6 -> 9
- net Row1: track 136.2 -> 128.6 mm, vias 8 -> 7
- net Col1: track 113.2 -> 118.9 mm
- net Col3: track 209.2 -> 214.3 mm
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