File: pcb/v2/roBa_R/roba_R.kicad_sch (KiCad schematic)
At the start: 50 parts, among them J2 Conn_01x01-Connector_Generic, J3 Conn_01x01-Connector_Generic, J4 Conn_01x01-Connector_Generic, J5 Conn_01x01-Connector_Generic, J6 Conn_01x01-Connector_Generic, J7 Conn_01x01-Connector_Generic, SW1 SW_PUSH, SW10 SW_PUSH, SW11 SW_PUSH, SW12 SW_PUSH, SW13 SW_PUSH, SW14 SW_PUSH, SW15 SW_PUSH, SW16 SW_PUSH, SW17 SW_PUSH, SW18 SW_PUSH, SW19 SW_PUSH, SW2 SW_PUSH, SW20 SW_PUSH, SW21 SW_SPDT, SW3 SW_PUSH, SW4 SW_PUSH, SW5 SW_PUSH, SW6 SW_PUSH, SW7 SW_PUSH, SW8 SW_PUSH, SW9 SW_PUSH

Commit message: Update schematics and PCBs
Parts:
- removed D20: D, roBa:Diode_SMD, symbol Device:D
- removed J1: ~, roBa:pmw3610_connector, symbol my:pmw3610_breakout
- removed SW20: SW_PUSH, roBa:SW_MX, symbol Switch:SW_Push
- added J8: ~, vik:vik-keyboard-connector-horizontal, symbol vik:vik-keyboard-connector
- D1, D10, D11, D12, D13, D14, D15, D16, D17, D18, D19, D2, D3, D4, D5, D6, D7, D8, D9: footprint roBa:Diode_SMD -> Diode_SMD:D_SOD-123
- SW1, SW10, SW11, SW13, SW14, SW15, SW17, SW18, SW19, SW2, SW3, SW4, SW5, SW6, SW7, SW8, SW9: footprint roBa:SW_MX -> roBa:gateron-ks27-choc-v1-mx-hotswap-curved-pads
- SW12, SW16: footprint roBa:SW_MX_Choc -> roBa:gateron-ks27-choc-v1-mx-hotswap-curved-pads
Connections:
- net CS: now also J8.10 (SPI_CS)
- net GND: now also J8.2 (GND)
- net MOTION: now also J8.8 (MOSI)
- net SCLK: now also J8.12 (SCLK)
- net SDIO: now also J8.11 (MISO)
- net 3.3V renamed +3.3V
- net +3.3V: now also J8.1 (3V3)
- net VCC: no longer names the net of U1.14 (5V)
- no-connect marks 11 -> 17
