File: pcb/pmw3610_breakout_for_roViBa/pmw3610_breakout_for_roViBa.kicad_sch (KiCad schematic)
At the start: 13 parts, among them J2 vik-module-connector, U1 MCP1700T-1802E/TT, U2 PMW3610

Commit message: Redo pmw3610 sensor board
Parts:
- C1: value 1uF -> 1u; LCSC (none) -> C14663
- C2: value 1uF -> 1u; LCSC (none) -> C15849
- C3, C8: value 100nF -> 100n; LCSC (none) -> C19666
- C4: value 10nF -> 10n; LCSC (none) -> C19666
- C5: value 100nF (X7R) -> 100n (X7R); LCSC (none) -> C19666
- C6: value 10uF (X7R) -> 10u (X7R); LCSC (none) -> C19666
- C7: value 10nF (X7R) -> 10n (X7R); LCSC (none) -> C19666
- C9: value 3.3uF/16V -> 3.3u/25V; LCSC (none) -> C19666
